Commit message: qawd

File: src/articubot_one/description/robot_core.xacro (robot description, xacro)
@@ -95,5 +95,5 @@
     <parent link="base_link"/>
     <child link="left_rear_wheel"/>
-    <origin xyz="-0.2 0.175 0" rpy="-${pi/2} 0 0"/>
+    <origin xyz="0.165 0.175 0" rpy="-${pi/2} 0 0"/>
     <axis xyz="0 0 1"/>
   </joint>
@@ -118,5 +118,5 @@
     <parent link="base_link"/>
     <child link="right_rear_wheel"/>
-    <origin xyz="-0.2 -0.175 0" rpy="${pi/2} 0 0"/>
+    <origin xyz="0.165 -0.175 0" rpy="${pi/2} 0 0"/>
     <axis xyz="0 0 -1"/>
   </joint>
